File: esp32-s2-mini-1/esp32-s2-mini-1.kicad_pcb (KiCad board)
At the start: 2 copper layers, 25.4 x 55.2 mm, 23 parts, among them J1 Conn_01x20_Male, J2 USB_C_Receptacle_USB2.0, J3 Conn_01x20_Male, U1 ESP32-S2-M, U2 LM1117-3.3

Commit message: Add signature and logos to the pcb back
Parts:
- added REF**: OSHW-Logo_5.7x6mm_SilkScreen, Designs:OSHW-Logo_5.7x6mm_SilkScreen, B.Cu at (154.2, 107.8)
- added REF**: KiCad-Logo_5mm_SilkScreen, Designs:KiCad-Logo_5mm_SilkScreen, B.Cu at (154.6, 118.8)
Other:
- board text added: "DESIGNED WITH"
- board text added: "by blurpy"
