File: esp32-s2-mini-1/esp32-s2-mini-1.kicad_sch (KiCad schematic)
At the start: 23 parts, among them J1 Conn_01x20_Male, J2 USB_C_Receptacle_USB2.0, J3 Conn_01x20_Male, U1 ESP32-S2-M, U2 LM1117-3.3

Commit message: Adding a title and date to the schematic
Other:
- title: (none) -> ESP32 S2 Mini Development Board
Changed lines of the file:
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@@
 (kicad_sch (version 20211123) (generator eeschema)
   (paper "A4")
+  (title_block
+    (title "ESP32 S2 Mini Development Board")
+    (date "2022-04-14")
+    (rev "1")
+  )
   (junction (at 229.87 41.91) (diameter 0) (color 0 0 0 0)
   )
